File: Elec/Light/mini_light.kicad_pcb (KiCad board)
At the start: 2 copper layers, 70 x 11.2 mm, 18 parts, among them J1 Conn_01x03, J2 Conn_01x03, U1 AL8860WT-7

Commit message: Update lib and pcb
Parts:
- D2, D3, D4, D5, D6, D7: footprint mini_light:LED_Cree-JE -> AM163:LED_Cree-JE
- J1, J2: value Conn_01x03 -> Conn_01x03_MountingPin
- L1: footprint mini_light:L_Bourns-SRN5040 -> AM163:L_Bourns-SRN5040
Connections:
- J1 pad MP: (no net) -> GND
- J2 pad MP: (no net) -> GND
Routing:
- net GND: vias 114 -> 109
